File: Hardware/Motor Driver/Motor Driver.kicad_sch (KiCad schematic)
At the start: 9 parts, among them J1 Conn_01x02, J2 Conn_01x02, J3 Conn_01x04, J4 Conn_01x04, J5 Conn_01x06, J6 Conn_01x06, J7 Conn_01x02

Commit message: Connected the battery and buck converter grounds, because isolation wasn't needed in this application.
Connections:
- net at J1.2 (Pin_2), J7.2 (Pin_2), U1.14 (GND)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: now also J2.2 (Pin_2), U1.8 (GND), U1.9 (GND), U2.8 (GND), U2.9 (GND)
Changed lines of the file:
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@@
+	)
+	(junction
+		(at 154.94 107.95)
+		(diameter 0)
+		(color 0 0 0 0)
 	)
 	(junction
@@
 	(wire
 		(pts
-			(xy 134.62 107.95) (xy 160.02 107.95)
+			(xy 134.62 107.95) (xy 154.94 107.95)
 		)
 		(stroke
@@
 	(wire
 		(pts
+			(xy 154.94 107.95) (xy 154.94 114.3)
+		)
+		(stroke
+			(width 0)
+			(type default)
+		)
+	)
+	(wire
+		(pts
 			(xy 66.04 95.25) (xy 66.04 91.44)
 		)
@@
 	(wire
 		(pts
+			(xy 154.94 107.95) (xy 160.02 107.95)
+		)
+		(stroke
+			(width 0)
+			(type default)
+		)
+	)
+	(wire
+		(pts
 			(xy 63.5 102.87) (xy 63.5 96.52)
 		)
@@
 	(wire
 		(pts
-			(xy 154.94 93.98) (xy 154.94 114.3)
-		)
-		(stroke
+			(xy 154.94 93.98) (xy 154.94 107.95)
+		)
+		(stroke
